File: kicad/kicad.kicad_pcb (KiCad board)
At the start: 2 copper layers, 68 x 34.5 mm, 61 parts, among them J1 USB_B_Micro, J3 swd, J5 led_front, J6 led_back, Q1 SI2365EDS-T1-GE3, Q2 2N7002, SW1 SW_Reed, SW2 Rotary_Encoder_Switch, SW3 SW_Push, U1 MCP73831-2-OT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

Commit message: rev1 pcb done
Parts:
- BZ1: moved to B.Cu
- moved C2 5.36 mm to (117.2, 74.5)
Routing:
- net led_en: track 11.4 -> 35.6 mm, vias 1 -> 2
- net GND: track 24.2 -> 30.7 mm, vias 5 -> 19
- net lcd_com: track 34.7 -> 36.9 mm
- net encoder_b: track 32.8 -> 34.5 mm
- net lcd_g2: track 23.4 -> 24.8 mm
- net lcd_d2: track 23.2 -> 24.3 mm
- net /vcc_en: track 7.89 -> 8.73 mm
- net lcd_e2: track 23.3 -> 24.1 mm
- net /vbat_prot: track 54.1 -> 53.9 mm, vias 6 -> 4
- added copper zone on B.Cu, net GND
Other:
- board size 68 x 34.5 mm -> 68 x 35.2 mm
- board text added: "+ -"
- board text added: "BikeoMeter V1 Anton Lööf 2021"
- board text added: "GND SWDCLK SWDIO"
- board text added: "GND VBAT"
- board text added: "REED"

Commit message: Rev2 psb with correct mcu size...
Parts:
- removed FB1: 1k@100M, Inductor_SMD:L_0603_1608Metric_Pad1.05x0.95mm_HandSolder
- C3: moved to B.Cu
- U2: footprint Package_QFP:LQFP-48_7x7mm_P0.5mm -> Package_DFN_QFN:QFN-48-1EP_7x7mm_P0.5mm_EP5.6x5.6mm
- moved TP1 17.3 mm to (126.8, 86.8)
- moved C4 10.8 mm to (141.5, 81.5), turned to 90 degrees
- moved C6 7.25 mm to (148.3, 91.7), turned to 180 degrees
- moved C8 7.19 mm to (143.8, 89.1), turned to 0 degrees
- moved C9 5.99 mm to (144.0, 81.9), turned to 0 degrees
- moved C3 4.10 mm to (149.2, 88.8), turned to 180 degrees
- moved C13 3.36 mm to (135.9, 100.1)
- moved C7 3.26 mm to (148.6, 86.3), turned to -90 degrees
- moved C5 2.77 mm to (143.8, 91.3), turned to 0 degrees
- moved R17 2.15 mm to (155.6, 77.7), turned to 0 degrees
- moved JP1 1.55 mm to (143.7, 93.4)
- moved U2 0.45 mm to (146.5, 86.8)
- moved D1 0.22 mm to (131.4, 77.7)
- moved R15 0.20 mm to (153.4, 83.3)
- moved L1 0.20 mm to (160.2, 89.7)
Connections:
- net Net-(C3-Pad1) renamed /vlcd
- net Net-(D2-Pad1) renamed /charge_stat
- net Net-(D2-Pad2) renamed /charge_ledr
- net Net-(R2-Pad1) renamed /charge_prog
- C8 pad 1: vcca -> vcc
- C9 pad 1: vcca -> vcc
- J1 pad 2: (no net) -> unconnected-(J1-Pad2)
- J1 pad 3: (no net) -> unconnected-(J1-Pad3)
- J1 pad 4: (no net) -> unconnected-(J1-Pad4)
- J1 pad 6: Net-(J1-Pad6) -> unconnected-(J1-Pad6)
- U2 pad 11: lcd_c2 -> reed_sw
- U2 pad 12: lcd_a3 -> led_en
- U2 pad 13: lcd_b3 -> lcd_a3
- U2 pad 15: beeper -> unconnected-(U2-Pad15)
- U2 pad 16: lcd_c3 -> lcd_b3
- U2 pad 17: lcd_d3 -> lcd_c3
- U2 pad 18: lcd_e3 -> lcd_d3
- U2 pad 19: lcd_g3 -> lcd_e3
- U2 pad 20: (no net) -> unconnected-(U2-Pad20)
- U2 pad 21: lcd_f3 -> lcd_g3
- U2 pad 22: lcd_1bc -> lcd_f3
- U2 pad 25: lcd_d2 -> lcd_1bc
- U2 pad 26: lcd_e2 -> beeper
- U2 pad 27: lcd_g2 -> lcd_e2
- U2 pad 28: (no net) -> lcd_d2
- U2 pad 3: (no net) -> encoder_b
- U2 pad 30: (no net) -> unconnected-(U2-Pad30)
- U2 pad 31: encoder_b -> led0
- U2 pad 32: encoder_a -> led1
- U2 pad 33: reed_sw -> led2
- U2 pad 38: (no net) -> lcd_g2
- U2 pad 4: (no net) -> encoder_a
- U2 pad 42: led_en -> unconnected-(U2-Pad42)
- U2 pad 43: led2 -> unconnected-(U2-Pad43)
- U2 pad 45: led1 -> lcd_c2
- U2 pad 46: led0 -> unconnected-(U2-Pad46)
- U2 pad 5: (no net) -> unconnected-(U2-Pad5)
- U2 pad 6: (no net) -> unconnected-(U2-Pad6)
- U2 pad 9: vcca -> vcc
Routing:
- net led0: track 36.7 -> 9.68 mm
- net led_en: track 35.6 -> 11.1 mm, vias 2 -> 0
- net led1: track 29.1 -> 9.02 mm
- net /nrst: track 53.8 -> 72.2 mm
- net lcd_com: track 36.9 -> 19.2 mm
- net vcc: track 78.7 -> 94.9 mm, vias 5 -> 6
- net encoder_b: track 34.5 -> 47.9 mm
- net encoder_a: track 37.8 -> 49.5 mm
- net unconnected-(J1-Pad6): track 0.00 -> 11.5 mm
- net Net-(J1-Pad6): track 11.5 -> 0.00 mm
- net lcd_g2: track 24.8 -> 14.2 mm
- net vcca: track 9.89 -> 0.00 mm, vias 1 -> 0
- net reed_sw: track 40.7 -> 31.6 mm, vias 1 -> 0
- net beeper: track 33.8 -> 25.5 mm
- net lcd_e2: track 24.1 -> 29.7 mm
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Other:
- net class Default removed
- rule pad_to_mask_clearance: 0.051 -> 0
- board text added: "BikeoMeter V2 Anton Lööf 2022"
- board text removed: "BikeoMeter V1 Anton Lööf 2021"
